Commit message: Rebase from 'upstream'

File: open_manipulator_description/ros2_control/omx.ros2_control.xacro (robot description, xacro)
@@ -103,6 +103,6 @@
         <param name="Position I Gain">100</param>
         <param name="Position D Gain">100</param>
-        <param name="Profile Velocity">11</param>
-        <param name="Profile Acceleration">2</param>
+        <param name="Profile Velocity">20</param>
+        <param name="Profile Acceleration">10</param>
         <param name="Drive Mode">4</param>
         <param name="Return Delay Time">0</param>
@@ -119,6 +119,6 @@
         <param name="Position I Gain">100</param>
         <param name="Position D Gain">100</param>
-        <param name="Profile Velocity">11</param>
-        <param name="Profile Acceleration">2</param>
+        <param name="Profile Velocity">20</param>
+        <param name="Profile Acceleration">10</param>
         <param name="Drive Mode">4</param>
         <param name="Return Delay Time">0</param>
@@ -135,6 +135,6 @@
         <param name="Position I Gain">100</param>
         <param name="Position D Gain">100</param>
-        <param name="Profile Velocity">11</param>
-        <param name="Profile Acceleration">2</param>
+        <param name="Profile Velocity">20</param>
+        <param name="Profile Acceleration">10</param>
         <param name="Drive Mode">4</param>
         <param name="Return Delay Time">0</param>
@@ -151,6 +151,6 @@
         <param name="Position I Gain">100</param>
         <param name="Position D Gain">100</param>
-        <param name="Profile Velocity">11</param>
-        <param name="Profile Acceleration">2</param>
+        <param name="Profile Velocity">20</param>
+        <param name="Profile Acceleration">10</param>
         <param name="Drive Mode">4</param>
         <param name="Return Delay Time">0</param>
@@ -164,6 +164,6 @@
         <state_interface name="Present Current"/>
         <param name="Operating Mode">5</param>
-        <param name="Profile Velocity">11</param>
-        <param name="Profile Acceleration">2</param>
+        <param name="Profile Velocity">20</param>
+        <param name="Profile Acceleration">10</param>
         <param name="Drive Mode">4</param>
         <param name="Return Delay Time">0</param>

File: open_manipulator_description/ros2_control/omy_3m_end_unit.ros2_control.xacro (robot description, xacro)
@@ -45,6 +45,4 @@
         <param name="SyncTable Write Size">12</param>
         <param name="SyncTable Enable">1</param>
-        <param name="Goal Velocity">2970</param>
-        <param name="Goal Current">661</param>
       </gpio>
     </ros2_control>

File: open_manipulator_description/ros2_control/omy_f3m.ros2_control.xacro (robot description, xacro)
@@ -91,7 +91,5 @@
         <state_interface name="Present Velocity"/>
         <state_interface name="Present Current"/>
-        <state_interface name="Torque Enable"/>
-        <state_interface name="Present Input Voltage"/>
-        <param name="Drive Mode">0</param>
+        <param name="Drive Mode">4</param>
         <param name="Velocity Limit">3591</param>
         <param name="Acceleration Limit">8050</param>
@@ -104,4 +102,6 @@
         <param name="Velocity I Gain">1565630</param>
         <param name="Operating Mode">3</param>
+        <param name="Profile Acceleration Time">13</param>
+        <param name="Profile Time">26</param>
       </gpio>
       <gpio name="dxl2">
@@ -112,7 +112,5 @@
         <state_interface name="Present Velocity"/>
         <state_interface name="Present Current"/>
-        <state_interface name="Torque Enable"/>
-        <state_interface name="Present Input Voltage"/>
-        <param name="Drive Mode">1</param>
+        <param name="Drive Mode">5</param>
         <param name="Velocity Limit">3591</param>
         <param name="Acceleration Limit">8050</param>
@@ -124,4 +122,6 @@
         <param name="Velocity I Gain">1565630</param>
         <param name="Operating Mode">3</param>
+        <param name="Profile Acceleration Time">13</param>
+        <param name="Profile Time">26</param>
       </gpio>
       <gpio name="dxl3">
@@ -132,16 +132,16 @@
         <state_interface name="Present Velocity"/>
         <state_interface name="Present Current"/>
-        <state_interface name="Torque Enable"/>
-        <state_interface name="Present Input Voltage"/>
-        <param name="Drive Mode">0</param>
-        <param name="Velocity Limit">6486</param>
-        <param name="Acceleration Limit">8050</param>
-        <param name="Profile Velocity">6486</param>
-        <param name="Profile Acceleration">8050</param>
-        <param name="Return Delay Time">0</param>
-        <param name="Position P Gain">1583185</param>
-        <param name="Velocity P Gain">18184</param>
-        <param name="Velocity I Gain">1585331</param>
-        <param name="Operating Mode">3</param>
+        <param name="Drive Mode">4</param>
+        <param name="Velocity Limit">6486</param>
+        <param name="Acceleration Limit">8050</param>
+        <param name="Profile Velocity">6486</param>
+        <param name="Profile Acceleration">8050</param>
+        <param name="Return Delay Time">0</param>
+        <param name="Position P Gain">1583185</param>
+        <param name="Velocity P Gain">18184</param>
+        <param name="Velocity I Gain">1585331</param>
+        <param name="Operating Mode">3</param>
+        <param name="Profile Acceleration Time">13</param>
+        <param name="Profile Time">26</param>
       </gpio>
       <gpio name="dxl4">
@@ -152,16 +152,16 @@
         <state_interface name="Present Velocity"/>
         <state_interface name="Present Current"/>
-        <state_interface name="Torque Enable"/>
-        <state_interface name="Present Input Voltage"/>
-        <param name="Drive Mode">1</param>
-        <param name="Velocity Limit">6486</param>
-        <param name="Acceleration Limit">8050</param>
-        <param name="Profile Velocity">6486</param>
-        <param name="Profile Acceleration">8050</param>
-        <param name="Return Delay Time">0</param>
-        <param name="Position P Gain">1583185</param>
-        <param name="Velocity P Gain">18184</param>
-        <param name="Velocity I Gain">1585331</param>
-        <param name="Operating Mode">3</param>
+        <param name="Drive Mode">5</param>
+        <param name="Velocity Limit">6486</param>
+        <param name="Acceleration Limit">8050</param>
+        <param name="Profile Velocity">6486</param>
+        <param name="Profile Acceleration">8050</param>
+        <param name="Return Delay Time">0</param>
+        <param name="Position P Gain">1583185</param>
+        <param name="Velocity P Gain">18184</param>
+        <param name="Velocity I Gain">1585331</param>
+        <param name="Operating Mode">3</param>
+        <param name="Profile Acceleration Time">13</param>
+        <param name="Profile Time">26</param>
       </gpio>
       <gpio name="dxl5">
@@ -172,16 +172,16 @@
         <state_interface name="Present Velocity"/>
         <state_interface name="Present Current"/>
-        <state_interface name="Torque Enable"/>
-        <state_interface name="Present Input Voltage"/>
-        <param name="Drive Mode">0</param>
-        <param name="Velocity Limit">6486</param>
-        <param name="Acceleration Limit">8050</param>
-        <param name="Profile Velocity">6486</param>
-        <param name="Profile Acceleration">8050</param>
-        <param name="Return Delay Time">0</param>
-        <param name="Position P Gain">1583185</param>
-        <param name="Velocity P Gain">18184</param>
-        <param name="Velocity I Gain">1585331</param>
-        <param name="Operating Mode">3</param>
+        <param name="Drive Mode">4</param>
+        <param name="Velocity Limit">6486</param>
+        <param name="Acceleration Limit">8050</param>
+        <param name="Profile Velocity">6486</param>
+        <param name="Profile Acceleration">8050</param>
+        <param name="Return Delay Time">0</param>
+        <param name="Position P Gain">1583185</param>
+        <param name="Velocity P Gain">18184</param>
+        <param name="Velocity I Gain">1585331</param>
+        <param name="Operating Mode">3</param>
+        <param name="Profile Acceleration Time">13</param>
+        <param name="Profile Time">26</param>
       </gpio>
       <gpio name="dxl6">
@@ -192,16 +192,16 @@
         <state_interface name="Present Velocity"/>
         <state_interface name="Present Current"/>
-        <state_interface name="Torque Enable"/>
-        <state_interface name="Present Input Voltage"/>
-        <param name="Drive Mode">1</param>
-        <param name="Velocity Limit">6486</param>
-        <param name="Acceleration Limit">8050</param>
-        <param name="Profile Velocity">6486</param>
-        <param name="Profile Acceleration">8050</param>
-        <param name="Return Delay Time">0</param>
-        <param name="Position P Gain">1583185</param>
-        <param name="Velocity P Gain">18184</param>
-        <param name="Velocity I Gain">1585331</param>
-        <param name="Operating Mode">3</param>
+        <param name="Drive Mode">5</param>
+        <param name="Velocity Limit">6486</param>
+        <param name="Acceleration Limit">8050</param>
+        <param name="Profile Velocity">6486</param>
+        <param name="Profile Acceleration">8050</param>
+        <param name="Return Delay Time">0</param>
+        <param name="Position P Gain">1583185</param>
+        <param name="Velocity P Gain">18184</param>
+        <param name="Velocity I Gain">1585331</param>
+        <param name="Operating Mode">3</param>
+        <param name="Profile Acceleration Time">13</param>
+        <param name="Profile Time">26</param>
       </gpio>
       <gpio name="omy_hat">

File: open_manipulator_description/ros2_control/omy_f3m_end_unit.ros2_control.xacro (robot description, xacro)
@@ -73,10 +73,22 @@
         </joint>
       </xacro:if>
-      <gpio name="omy_end">
+      <gpio name="dxl7">
         <command_interface name="Goal Position"/>
         <state_interface name="Present Position"/>
         <state_interface name="Present Velocity"/>
         <state_interface name="Present Current"/>
-        <param name="type">dxl</param>
+        <param name="type">virtual_dxl</param>
+        <param name="ID">7</param>
+        <param name="model_num">231</param>
+        <param name="comm_id">210</param>
+        <param name="Goal Velocity">2970</param>
+        <param name="Goal Current">661</param>
+      </gpio>
+      <gpio name="omy_end">
+        <!-- <command_interface name="R LED"/>
+        <command_interface name="G LED"/>
+        <command_interface name="B LED"/> -->
+        <state_interface name="Button Status"/>
+        <param name="type">controller</param>
         <param name="ID">210</param>
         <param name="Baud Rate (Bus)">6</param>
@@ -93,6 +105,4 @@
         <param name="SyncTable Write Size">12</param>
         <param name="SyncTable Enable">1</param>
-        <param name="Goal Velocity">2970</param>
-        <param name="Goal Current">661</param>
       </gpio>
     </ros2_control>

File: open_manipulator_description/ros2_control/omy_f3m_smooth.ros2_control.xacro (robot description, xacro)
@@ -1,5 +1,5 @@
 <?xml version="1.0"?>
 <robot xmlns:xacro="http://www.ros.org/wiki/xacro">
-  <xacro:macro name="omy_3m_system" params="name prefix port_name:=^|/dev/ttyAMA2 use_sim:=^|false use_fake_hardware:=^|false fake_sensor_commands:=^|false">
+  <xacro:macro name="omy_f3m_system" params="name prefix port_name:=^|/dev/ttyAMA2 use_sim:=^|false use_fake_hardware:=^|false fake_sensor_commands:=^|false">
     <ros2_control name="${name}" type="system" is_async="true">
       <xacro:if value="$(arg use_sim)">
@@ -102,6 +102,6 @@
         <param name="Velocity I Gain">1565630</param>
         <param name="Operating Mode">3</param>
-        <param name="Profile Acceleration Time">13</param>
-        <param name="Profile Time">26</param>
+        <param name="Profile Acceleration Time">250</param>
+        <param name="Profile Time">500</param>
       </gpio>
       <gpio name="dxl2">
@@ -122,6 +122,6 @@
         <param name="Velocity I Gain">1565630</param>
         <param name="Operating Mode">3</param>
-        <param name="Profile Acceleration Time">13</param>
-        <param name="Profile Time">26</param>
+        <param name="Profile Acceleration Time">250</param>
+        <param name="Profile Time">500</param>
       </gpio>
       <gpio name="dxl3">
@@ -142,6 +142,6 @@
         <param name="Velocity I Gain">1585331</param>
         <param name="Operating Mode">3</param>
-        <param name="Profile Acceleration Time">13</param>
-        <param name="Profile Time">26</param>
+        <param name="Profile Acceleration Time">250</param>
+        <param name="Profile Time">500</param>
       </gpio>
       <gpio name="dxl4">
@@ -162,6 +162,6 @@
         <param name="Velocity I Gain">1585331</param>
         <param name="Operating Mode">3</param>
-        <param name="Profile Acceleration Time">13</param>
-        <param name="Profile Time">26</param>
+        <param name="Profile Acceleration Time">250</param>
+        <param name="Profile Time">500</param>
       </gpio>
       <gpio name="dxl5">
@@ -182,6 +182,6 @@
         <param name="Velocity I Gain">1585331</param>
         <param name="Operating Mode">3</param>
-        <param name="Profile Acceleration Time">13</param>
-        <param name="Profile Time">26</param>
+        <param name="Profile Acceleration Time">250</param>
+        <param name="Profile Time">500</param>
       </gpio>
       <gpio name="dxl6">
@@ -202,6 +202,6 @@
         <param name="Velocity I Gain">1585331</param>
         <param name="Operating Mode">3</param>
-        <param name="Profile Acceleration Time">13</param>
-        <param name="Profile Time">26</param>
+        <param name="Profile Acceleration Time">250</param>
+        <param name="Profile Time">500</param>
       </gpio>
       <gpio name="omy_hat">

File: open_manipulator_description/urdf/omx/omx.urdf.xacro (robot description, xacro)
@@ -6,7 +6,8 @@
   <xacro:arg name="fake_sensor_commands" default="false" />
   <xacro:arg name="port_name" default="/dev/ttyUSB0" />
+  <xacro:arg name="ros2_control_type" default="omx" />
   <xacro:include filename="$(find open_manipulator_description)/gazebo/omx.gazebo.xacro" />
   <xacro:include filename="$(find open_manipulator_description)/urdf/omx/omx_arm.urdf.xacro" />
-  <xacro:include filename="$(find open_manipulator_description)/ros2_control/omx.ros2_control.xacro" />
+  <xacro:include filename="$(find open_manipulator_description)/ros2_control/$(arg ros2_control_type).ros2_control.xacro" />
   <link name="world"/>
   <joint name="$(arg prefix)world_fixed" type="fixed">

File: open_manipulator_description/urdf/omy_3m/omy_3m.urdf.xacro (robot description, xacro)
@@ -5,7 +5,8 @@
   <xacro:arg name="use_fake_hardware" default="false" />
   <xacro:arg name="fake_sensor_commands" default="false" />
+  <xacro:arg name="ros2_control_type" default="omy_3m" />
   <xacro:include filename="$(find open_manipulator_description)/urdf/omy_3m/omy_3m_arm.urdf.xacro" />
   <xacro:include filename="$(find open_manipulator_description)/gazebo/omy_3m.gazebo.xacro" />
-  <xacro:include filename="$(find open_manipulator_description)/ros2_control/omy_3m.ros2_control.xacro" />
+  <xacro:include filename="$(find open_manipulator_description)/ros2_control/$(arg ros2_control_type).ros2_control.xacro" />
   <xacro:include filename="$(find open_manipulator_description)/ros2_control/omy_3m_end_unit.ros2_control.xacro" />
   <link name="world"/>

File: open_manipulator_description/urdf/omy_f3m/omy_f3m.urdf.xacro (robot description, xacro)
@@ -6,9 +6,10 @@
   <xacro:arg name="fake_sensor_commands" default="false" />
   <xacro:arg name="config_type" default="omy_f3m" />
+  <xacro:arg name="ros2_control_type" default="omy_f3m" />
   <xacro:include filename="$(find open_manipulator_description)/urdf/omy_f3m/omy_f3m_arm.urdf.xacro" />
   <xacro:include filename="$(find open_manipulator_description)/gazebo/omy_f3m.gazebo.xacro" />
   <xacro:include filename="$(find open_manipulator_description)/urdf/omy_f3m/rh_p12_rn_a.urdf.xacro" />
   <xacro:include filename="$(find open_manipulator_description)/gazebo/rh_p12_rn_a.gazebo.xacro" />
-  <xacro:include filename="$(find open_manipulator_description)/ros2_control/omy_f3m.ros2_control.xacro" />
+  <xacro:include filename="$(find open_manipulator_description)/ros2_control/$(arg ros2_control_type).ros2_control.xacro" />
   <xacro:include filename="$(find open_manipulator_description)/ros2_control/omy_f3m_end_unit.ros2_control.xacro" />
   <link name="world"/>

File: open_manipulator_description/urdf/omy_l100/omy_l100.urdf.xacro (robot description, xacro)
@@ -6,7 +6,8 @@
   <xacro:arg name="fake_sensor_commands" default="false" />
   <xacro:arg name="port_name" default="/dev/ttyUSB0" />
+  <xacro:arg name="ros2_control_type" default="omy_l100" />
   <xacro:include filename="$(find open_manipulator_description)/urdf/omy_l100/omy_l100_arm.urdf" />
   <xacro:include filename="$(find open_manipulator_description)/gazebo/omy_l100.gazebo.xacro" />
-  <xacro:include filename="$(find open_manipulator_description)/ros2_control/omy_l100.ros2_control.xacro" />
+  <xacro:include filename="$(find open_manipulator_description)/ros2_control/$(arg ros2_control_type).ros2_control.xacro" />
   <link name="world"/>
   <joint name="$(arg prefix)world_fixed" type="fixed">
