Commit message: Rebase from 'upstream'

File: open_manipulator_description/ros2_control/omy_3m.ros2_control.xacro (robot description, xacro)
@@ -102,6 +102,6 @@
         <param name="Velocity I Gain">1565630</param>
         <param name="Operating Mode">3</param>
-        <param name="Profile Acceleration Time">13</param>
-        <param name="Profile Time">26</param>
+        <param name="Profile Acceleration Time">20</param>
+        <param name="Profile Time">40</param>
       </gpio>
       <gpio name="dxl2">
@@ -122,6 +122,6 @@
         <param name="Velocity I Gain">1565630</param>
         <param name="Operating Mode">3</param>
-        <param name="Profile Acceleration Time">13</param>
-        <param name="Profile Time">26</param>
+        <param name="Profile Acceleration Time">20</param>
+        <param name="Profile Time">40</param>
       </gpio>
       <gpio name="dxl3">
@@ -142,6 +142,6 @@
         <param name="Velocity I Gain">1585331</param>
         <param name="Operating Mode">3</param>
-        <param name="Profile Acceleration Time">13</param>
-        <param name="Profile Time">26</param>
+        <param name="Profile Acceleration Time">20</param>
+        <param name="Profile Time">40</param>
       </gpio>
       <gpio name="dxl4">
@@ -162,6 +162,6 @@
         <param name="Velocity I Gain">1585331</param>
         <param name="Operating Mode">3</param>
-        <param name="Profile Acceleration Time">13</param>
-        <param name="Profile Time">26</param>
+        <param name="Profile Acceleration Time">20</param>
+        <param name="Profile Time">40</param>
       </gpio>
       <gpio name="dxl5">
@@ -182,6 +182,6 @@
         <param name="Velocity I Gain">1585331</param>
         <param name="Operating Mode">3</param>
-        <param name="Profile Acceleration Time">13</param>
-        <param name="Profile Time">26</param>
+        <param name="Profile Acceleration Time">20</param>
+        <param name="Profile Time">40</param>
       </gpio>
       <gpio name="dxl6">
@@ -202,6 +202,6 @@
         <param name="Velocity I Gain">1585331</param>
         <param name="Operating Mode">3</param>
-        <param name="Profile Acceleration Time">13</param>
-        <param name="Profile Time">26</param>
+        <param name="Profile Acceleration Time">20</param>
+        <param name="Profile Time">40</param>
       </gpio>
       <gpio name="omy_hat">

File: open_manipulator_description/ros2_control/omy_f3m.ros2_control.xacro (robot description, xacro)
@@ -102,6 +102,6 @@
         <param name="Velocity I Gain">1565630</param>
         <param name="Operating Mode">3</param>
-        <param name="Profile Acceleration Time">13</param>
-        <param name="Profile Time">26</param>
+        <param name="Profile Acceleration Time">20</param>
+        <param name="Profile Time">40</param>
       </gpio>
       <gpio name="dxl2">
@@ -122,6 +122,6 @@
         <param name="Velocity I Gain">1565630</param>
         <param name="Operating Mode">3</param>
-        <param name="Profile Acceleration Time">13</param>
-        <param name="Profile Time">26</param>
+        <param name="Profile Acceleration Time">20</param>
+        <param name="Profile Time">40</param>
       </gpio>
       <gpio name="dxl3">
@@ -142,6 +142,6 @@
         <param name="Velocity I Gain">1585331</param>
         <param name="Operating Mode">3</param>
-        <param name="Profile Acceleration Time">13</param>
-        <param name="Profile Time">26</param>
+        <param name="Profile Acceleration Time">20</param>
+        <param name="Profile Time">40</param>
       </gpio>
       <gpio name="dxl4">
@@ -162,6 +162,6 @@
         <param name="Velocity I Gain">1585331</param>
         <param name="Operating Mode">3</param>
-        <param name="Profile Acceleration Time">13</param>
-        <param name="Profile Time">26</param>
+        <param name="Profile Acceleration Time">20</param>
+        <param name="Profile Time">40</param>
       </gpio>
       <gpio name="dxl5">
@@ -182,6 +182,6 @@
         <param name="Velocity I Gain">1585331</param>
         <param name="Operating Mode">3</param>
-        <param name="Profile Acceleration Time">13</param>
-        <param name="Profile Time">26</param>
+        <param name="Profile Acceleration Time">20</param>
+        <param name="Profile Time">40</param>
       </gpio>
       <gpio name="dxl6">
@@ -202,6 +202,6 @@
         <param name="Velocity I Gain">1585331</param>
         <param name="Operating Mode">3</param>
-        <param name="Profile Acceleration Time">13</param>
-        <param name="Profile Time">26</param>
+        <param name="Profile Acceleration Time">20</param>
+        <param name="Profile Time">40</param>
       </gpio>
       <gpio name="omy_hat">

File: open_manipulator_description/urdf/omy_f3m/omy_f3m_arm.urdf.xacro (robot description, xacro)
@@ -106,5 +106,5 @@
             <origin xyz="0 0.125 0.08" rpy="0 0 0" />
             <geometry>
-               <cylinder radius="0.042" length="0.19"/>
+               <cylinder radius="0.042" length="0.17"/>
             </geometry>
          </collision>
@@ -196,5 +196,5 @@
             <origin xyz="0 -0.1 0" rpy="1.57 0 0" />
             <geometry>
-               <cylinder radius="0.09" length="0.22"/>
+               <cylinder radius="0.08" length="0.22"/>
             </geometry>
          </collision>
@@ -223,5 +223,5 @@
             <origin xyz="0 0.03 0.04" rpy="0 0 0" />
             <geometry>
-               <cylinder radius="0.04" length="0.12"/>
+               <cylinder radius="0.035" length="0.12"/>
             </geometry>
          </collision>
