Commit message: Rebase from 'release/jazzy/open_manipulator_description'

File: ros2_control/omx_f.ros2_control.xacro (robot description, xacro)
@@ -1,5 +1,5 @@
 <?xml version="1.0"?>
 <robot xmlns:xacro="http://www.ros.org/wiki/xacro">
-  <xacro:macro name="omy_f3m_system" params="name prefix port_name:=^|/dev/ttyAMA2 use_sim:=^|false use_fake_hardware:=^|false fake_sensor_commands:=^|false">
+  <xacro:macro name="omx_f_system" params="name prefix port_name:=^|/dev/ttyACM1 use_sim:=^|false use_fake_hardware:=^|false fake_sensor_commands:=^|false">
     <ros2_control name="${name}" type="system" is_async="true">
       <xacro:if value="$(arg use_sim)">
@@ -18,5 +18,5 @@
             <plugin>dynamixel_hardware_interface/DynamixelHardware</plugin>
             <param name="port_name">${port_name}</param>
-            <param name="baud_rate">6250000</param>
+            <param name="baud_rate">1000000</param>
             <param name="error_timeout_ms">500</param>
             <param name="dynamixel_model_folder">/param/dxl_model</param>
@@ -52,5 +52,4 @@
         <state_interface name="position"/>
         <state_interface name="velocity"/>
-        <state_interface name="effort"/>
       </joint>
       <joint name="${prefix}joint2">
@@ -58,5 +57,4 @@
         <state_interface name="position"/>
         <state_interface name="velocity"/>
-        <state_interface name="effort"/>
       </joint>
       <joint name="${prefix}joint3">
@@ -64,5 +62,4 @@
         <state_interface name="position"/>
         <state_interface name="velocity"/>
-        <state_interface name="effort"/>
       </joint>
       <joint name="${prefix}joint4">
@@ -70,5 +67,4 @@
         <state_interface name="position"/>
         <state_interface name="velocity"/>
-        <state_interface name="effort"/>
       </joint>
       <joint name="${prefix}joint5">
@@ -76,144 +72,119 @@
         <state_interface name="position"/>
         <state_interface name="velocity"/>
-        <state_interface name="effort"/>
       </joint>
-      <joint name="${prefix}joint6">
+      <joint name="${prefix}gripper_joint_1">
         <command_interface name="position"/>
         <state_interface name="position"/>
         <state_interface name="velocity"/>
-        <state_interface name="effort"/>
       </joint>
-      <gpio name="dxl1">
+      <xacro:if value="$(arg use_sim)">
+        <joint name="${prefix}gripper_joint_2">
+          <param name="mimic">${prefix}gripper_joint_1</param>
+          <param name="multiplier">-1</param>
+          <state_interface name="position"/>
+          <state_interface name="velocity"/>
+          <state_interface name="effort"/>
+        </joint>
+      </xacro:if>
+      <gpio name="dxl11">
         <param name="type">dxl</param>
-        <param name="ID">1</param>
+        <param name="ID">11</param>
         <command_interface name="Goal Position"/>
         <state_interface name="Present Position"/>
         <state_interface name="Present Velocity"/>
-        <state_interface name="Present Current"/>
         <param name="Drive Mode">4</param>
-        <param name="Velocity Limit">3591</param>
-        <param name="Acceleration Limit">8050</param>
-        <param name="Profile Velocity">3591</param>
-        <param name="Profile Acceleration">8050</param>
-        <param name="Homing Offset">0</param>
+        <param name="Operating Mode">4</param>
         <param name="Return Delay Time">0</param>
-        <param name="Position P Gain">1583185</param>
-        <param name="Velocity P Gain">41387</param>
-        <param name="Velocity I Gain">1565630</param>
-        <param name="Operating Mode">3</param>
-        <param name="Profile Acceleration Time">500</param>
-        <param name="Profile Time">1000</param>
+        <param name="Position P Gain">1000</param>
+        <param name="Position I Gain">0</param>
+        <param name="Position D Gain">1000</param>
+        <param name="Profile Velocity">50</param>
+        <param name="Profile Acceleration">25</param>
       </gpio>
-      <gpio name="dxl2">
+      <gpio name="dxl12">
         <param name="type">dxl</param>
-        <param name="ID">2</param>
+        <param name="ID">12</param>
         <command_interface name="Goal Position"/>
         <state_interface name="Present Position"/>
         <state_interface name="Present Velocity"/>
-        <state_interface name="Present Current"/>
-        <param name="Drive Mode">5</param>
-        <param name="Velocity Limit">3591</param>
-        <param name="Acceleration Limit">8050</param>
-        <param name="Profile Velocity">3591</param>
-        <param name="Profile Acceleration">8050</param>
+        <param name="Drive Mode">4</param>
+        <param name="Operating Mode">3</param>
         <param name="Return Delay Time">0</param>
-        <param name="Position P Gain">1583185</param>
-        <param name="Velocity P Gain">41387</param>
-        <param name="Velocity I Gain">1565630</param>
-        <param name="Operating Mode">3</param>
-        <param name="Profile Acceleration Time">500</param>
-        <param name="Profile Time">1000</param>
+        <param name="Min Position Limit">830</param>
+        <param name="Max Position Limit">3129</param>
+        <param name="Position P Gain">1000</param>
+        <param name="Position I Gain">0</param>
+        <param name="Position D Gain">1000</param>
+        <param name="Profile Velocity">50</param>
+        <param name="Profile Acceleration">25</param>
       </gpio>
-      <gpio name="dxl3">
+      <gpio name="dxl13">
         <param name="type">dxl</param>
-        <param name="ID">3</param>
+        <param name="ID">13</param>
         <command_interface name="Goal Position"/>
         <state_interface name="Present Position"/>
         <state_interface name="Present Velocity"/>
-        <state_interface name="Present Current"/>
         <param name="Drive Mode">4</param>
-        <param name="Velocity Limit">6486</param>
-        <param name="Acceleration Limit">8050</param>
-        <param name="Profile Velocity">6486</param>
-        <param name="Profile Acceleration">8050</param>
+        <param name="Operating Mode">3</param>
         <param name="Return Delay Time">0</param>
-        <param name="Position P Gain">1583185</param>
-        <param name="Velocity P Gain">18184</param>
-        <param name="Velocity I Gain">1585331</param>
-        <param name="Operating Mode">3</param>
-        <param name="Profile Acceleration Time">500</param>
-        <param name="Profile Time">1000</param>
+        <param name="Min Position Limit">1024</param>
+        <param name="Max Position Limit">3140</param>
+        <param name="Position P Gain">1000</param>
+        <param name="Position I Gain">0</param>
+        <param name="Position D Gain">1000</param>
+        <param name="Profile Velocity">50</param>
+        <param name="Profile Acceleration">25</param>
       </gpio>
-      <gpio name="dxl4">
+      <gpio name="dxl14">
         <param name="type">dxl</param>
-        <param name="ID">4</param>
+        <param name="ID">14</param>
         <command_interface name="Goal Position"/>
         <state_interface name="Present Position"/>
         <state_interface name="Present Velocity"/>
-        <state_interface name="Present Current"/>
-        <param name="Drive Mode">5</param>
-        <param name="Velocity Limit">6486</param>
-        <param name="Acceleration Limit">8050</param>
-        <param name="Profile Velocity">6486</param>
-        <param name="Profile Acceleration">8050</param>
+        <param name="Drive Mode">4</param>
+        <param name="Operating Mode">3</param>
         <param name="Return Delay Time">0</param>
-        <param name="Position P Gain">1583185</param>
-        <param name="Velocity P Gain">18184</param>
-        <param name="Velocity I Gain">1585331</param>
-        <param name="Operating Mode">3</param>
-        <param name="Profile Acceleration Time">500</param>
-        <param name="Profile Time">1000</param>
+        <param name="Min Position Limit">0</param>
+        <param name="Max Position Limit">4095</param>
+        <param name="Position P Gain">1000</param>
+        <param name="Position I Gain">0</param>
+        <param name="Position D Gain">1000</param>
+        <param name="Profile Velocity">50</param>
+        <param name="Profile Acceleration">25</param>
       </gpio>
-      <gpio name="dxl5">
+      <gpio name="dxl15">
         <param name="type">dxl</param>
-        <param name="ID">5</param>
+        <param name="ID">15</param>
         <command_interface name="Goal Position"/>
         <state_interface name="Present Position"/>
         <state_interface name="Present Velocity"/>
-        <state_interface name="Present Current"/>
         <param name="Drive Mode">4</param>
-        <param name="Velocity Limit">6486</param>
-        <param name="Acceleration Limit">8050</param>
-        <param name="Profile Velocity">6486</param>
-        <param name="Profile Acceleration">8050</param>
+        <param name="Operating Mode">3</param>
         <param name="Return Delay Time">0</param>
-        <param name="Position P Gain">1583185</param>
-        <param name="Velocity P Gain">18184</param>
-        <param name="Velocity I Gain">1585331</param>
-        <param name="Operating Mode">3</param>
-        <param name="Profile Acceleration Time">500</param>
-        <param name="Profile Time">1000</param>
+        <param name="Min Position Limit">0</param>
+        <param name="Max Position Limit">4095</param>
+        <param name="Position P Gain">1000</param>
+        <param name="Position I Gain">0</param>
+        <param name="Position D Gain">1000</param>
+        <param name="Profile Velocity">50</param>
+        <param name="Profile Acceleration">25</param>
       </gpio>
-      <gpio name="dxl6">
+      <gpio name="dxl16">
         <param name="type">dxl</param>
-        <param name="ID">6</param>
+        <param name="ID">16</param>
         <command_interface name="Goal Position"/>
         <state_interface name="Present Position"/>
         <state_interface name="Present Velocity"/>
-        <state_interface name="Present Current"/>
-        <param name="Drive Mode">5</param>
-        <param name="Velocity Limit">6486</param>
-        <param name="Acceleration Limit">8050</param>
-        <param name="Profile Velocity">6486</param>
-        <param name="Profile Acceleration">8050</param>
+        <param name="Drive Mode">4</param>
+        <param name="Operating Mode">5</param>
         <param name="Return Delay Time">0</param>
-        <param name="Position P Gain">1583185</param>
-        <param name="Velocity P Gain">18184</param>
-        <param name="Velocity I Gain">1585331</param>
-        <param name="Operating Mode">3</param>
-        <param name="Profile Acceleration Time">500</param>
-        <param name="Profile Time">1000</param>
-      </gpio>
-      <gpio name="omy_hat">
-        <param name="type">controller</param>
-        <param name="ID">200</param>
-        <param name="Power Enable">1</param>
-        <param name="Voltage Control Enable">1</param>
-        <param name="R LED">200</param>
-        <param name="G LED">200</param>
-        <param name="B LED">120</param>
-        <param name="Baud Rate (Bus)">8</param>
-        <param name="DXL Baud Rate">8</param>
-        <param name="Status">0</param>
+        <param name="Position P Gain">1000</param>
+        <param name="Position I Gain">0</param>
+        <param name="Position D Gain">1000</param>
+        <param name="Profile Velocity">50</param>
+        <param name="Profile Acceleration">25</param>
+        <param name="Current Limit">600</param>
+        <param name="Goal Current">600</param>
+        <param name="Shutdown">21</param>
       </gpio>
     </ros2_control>

File: ros2_control/omy_f3m_current.ros2_control.xacro (robot description, xacro)
@@ -49,5 +49,5 @@
       </xacro:unless>
       <joint name="${prefix}joint1">
-        <command_interface name="position"/>
+        <command_interface name="effort"/>
         <state_interface name="position"/>
         <state_interface name="velocity"/>
@@ -55,5 +55,5 @@
       </joint>
       <joint name="${prefix}joint2">
-        <command_interface name="position"/>
+        <command_interface name="effort"/>
         <state_interface name="position"/>
         <state_interface name="velocity"/>
@@ -61,5 +61,5 @@
       </joint>
       <joint name="${prefix}joint3">
-        <command_interface name="position"/>
+        <command_interface name="effort"/>
         <state_interface name="position"/>
         <state_interface name="velocity"/>
@@ -67,5 +67,5 @@
       </joint>
       <joint name="${prefix}joint4">
-        <command_interface name="position"/>
+        <command_interface name="effort"/>
         <state_interface name="position"/>
         <state_interface name="velocity"/>
@@ -73,5 +73,5 @@
       </joint>
       <joint name="${prefix}joint5">
-        <command_interface name="position"/>
+        <command_interface name="effort"/>
         <state_interface name="position"/>
         <state_interface name="velocity"/>
@@ -79,5 +79,5 @@
       </joint>
       <joint name="${prefix}joint6">
-        <command_interface name="position"/>
+        <command_interface name="effort"/>
         <state_interface name="position"/>
         <state_interface name="velocity"/>
@@ -87,8 +87,9 @@
         <param name="type">dxl</param>
         <param name="ID">1</param>
-        <command_interface name="Goal Position"/>
-        <state_interface name="Present Position"/>
-        <state_interface name="Present Velocity"/>
-        <state_interface name="Present Current"/>
+        <command_interface name="Goal Current"/>
+        <state_interface name="Present Position"/>
+        <state_interface name="Present Velocity"/>
+        <state_interface name="Present Current"/>
+        <param name="Torque Enable">1</param>
         <param name="Drive Mode">4</param>
         <param name="Velocity Limit">3591</param>
@@ -101,15 +102,17 @@
         <param name="Velocity P Gain">41387</param>
         <param name="Velocity I Gain">1565630</param>
-        <param name="Operating Mode">3</param>
-        <param name="Profile Acceleration Time">500</param>
-        <param name="Profile Time">1000</param>
+        <param name="Operating Mode">0</param>
+        <param name="Profile Acceleration Time">20</param>
+        <param name="Profile Time">40</param>
+        <param name="Bus Watchdog">1</param>
       </gpio>
       <gpio name="dxl2">
         <param name="type">dxl</param>
         <param name="ID">2</param>
-        <command_interface name="Goal Position"/>
-        <state_interface name="Present Position"/>
-        <state_interface name="Present Velocity"/>
-        <state_interface name="Present Current"/>
+        <command_interface name="Goal Current"/>
+        <state_interface name="Present Position"/>
+        <state_interface name="Present Velocity"/>
+        <state_interface name="Present Current"/>
+        <param name="Torque Enable">1</param>
         <param name="Drive Mode">5</param>
         <param name="Velocity Limit">3591</param>
@@ -121,15 +124,17 @@
         <param name="Velocity P Gain">41387</param>
         <param name="Velocity I Gain">1565630</param>
-        <param name="Operating Mode">3</param>
-        <param name="Profile Acceleration Time">500</param>
-        <param name="Profile Time">1000</param>
+        <param name="Operating Mode">0</param>
+        <param name="Profile Acceleration Time">20</param>
+        <param name="Profile Time">40</param>
+        <param name="Bus Watchdog">1</param>
       </gpio>
       <gpio name="dxl3">
         <param name="type">dxl</param>
         <param name="ID">3</param>
-        <command_interface name="Goal Position"/>
-        <state_interface name="Present Position"/>
-        <state_interface name="Present Velocity"/>
-        <state_interface name="Present Current"/>
+        <command_interface name="Goal Current"/>
+        <state_interface name="Present Position"/>
+        <state_interface name="Present Velocity"/>
+        <state_interface name="Present Current"/>
+        <param name="Torque Enable">1</param>
         <param name="Drive Mode">4</param>
         <param name="Velocity Limit">6486</param>
@@ -141,15 +146,17 @@
         <param name="Velocity P Gain">18184</param>
         <param name="Velocity I Gain">1585331</param>
-        <param name="Operating Mode">3</param>
-        <param name="Profile Acceleration Time">500</param>
-        <param name="Profile Time">1000</param>
+        <param name="Operating Mode">0</param>
+        <param name="Profile Acceleration Time">20</param>
+        <param name="Profile Time">40</param>
+        <param name="Bus Watchdog">1</param>
       </gpio>
       <gpio name="dxl4">
         <param name="type">dxl</param>
         <param name="ID">4</param>
-        <command_interface name="Goal Position"/>
-        <state_interface name="Present Position"/>
-        <state_interface name="Present Velocity"/>
-        <state_interface name="Present Current"/>
+        <command_interface name="Goal Current"/>
+        <state_interface name="Present Position"/>
+        <state_interface name="Present Velocity"/>
+        <state_interface name="Present Current"/>
+        <param name="Torque Enable">1</param>
         <param name="Drive Mode">5</param>
         <param name="Velocity Limit">6486</param>
@@ -161,15 +168,17 @@
         <param name="Velocity P Gain">18184</param>
         <param name="Velocity I Gain">1585331</param>
-        <param name="Operating Mode">3</param>
-        <param name="Profile Acceleration Time">500</param>
-        <param name="Profile Time">1000</param>
+        <param name="Operating Mode">0</param>
+        <param name="Profile Acceleration Time">20</param>
+        <param name="Profile Time">40</param>
+        <param name="Bus Watchdog">1</param>
       </gpio>
       <gpio name="dxl5">
         <param name="type">dxl</param>
         <param name="ID">5</param>
-        <command_interface name="Goal Position"/>
-        <state_interface name="Present Position"/>
-        <state_interface name="Present Velocity"/>
-        <state_interface name="Present Current"/>
+        <command_interface name="Goal Current"/>
+        <state_interface name="Present Position"/>
+        <state_interface name="Present Velocity"/>
+        <state_interface name="Present Current"/>
+        <param name="Torque Enable">1</param>
         <param name="Drive Mode">4</param>
         <param name="Velocity Limit">6486</param>
@@ -181,15 +190,17 @@
         <param name="Velocity P Gain">18184</param>
         <param name="Velocity I Gain">1585331</param>
-        <param name="Operating Mode">3</param>
-        <param name="Profile Acceleration Time">500</param>
-        <param name="Profile Time">1000</param>
+        <param name="Operating Mode">0</param>
+        <param name="Profile Acceleration Time">20</param>
+        <param name="Profile Time">40</param>
+        <param name="Bus Watchdog">1</param>
       </gpio>
       <gpio name="dxl6">
         <param name="type">dxl</param>
         <param name="ID">6</param>
-        <command_interface name="Goal Position"/>
-        <state_interface name="Present Position"/>
-        <state_interface name="Present Velocity"/>
-        <state_interface name="Present Current"/>
+        <command_interface name="Goal Current"/>
+        <state_interface name="Present Position"/>
+        <state_interface name="Present Velocity"/>
+        <state_interface name="Present Current"/>
+        <param name="Torque Enable">1</param>
         <param name="Drive Mode">5</param>
         <param name="Velocity Limit">6486</param>
@@ -201,7 +212,8 @@
         <param name="Velocity P Gain">18184</param>
         <param name="Velocity I Gain">1585331</param>
-        <param name="Operating Mode">3</param>
-        <param name="Profile Acceleration Time">500</param>
-        <param name="Profile Time">1000</param>
+        <param name="Operating Mode">0</param>
+        <param name="Profile Acceleration Time">20</param>
+        <param name="Profile Time">40</param>
+        <param name="Bus Watchdog">1</param>
       </gpio>
       <gpio name="omy_hat">
