Commit message: Rebase from 'release/jazzy/open_manipulator_description'

File: ros2_control/omy_l100_position.ros2_control.xacro (robot description, xacro)
@@ -1,6 +1,6 @@
 <?xml version="1.0"?>
 <robot xmlns:xacro="http://www.ros.org/wiki/xacro">
-  <xacro:macro name="omy_f3m_system" params="name prefix port_name:=^|/dev/ttyAMA2 use_sim:=^|false use_fake_hardware:=^|false fake_sensor_commands:=^|false">
-    <ros2_control name="${name}" type="system" is_async="true">
+  <xacro:macro name="omy_l100_system" params="name prefix port_name:=^|/dev/ttyUSB0 use_sim:=^|false use_fake_hardware:=^|false fake_sensor_commands:=^|false">
+    <ros2_control name="${name}" type="system">
       <xacro:if value="$(arg use_sim)">
         <hardware>
@@ -18,25 +18,27 @@
             <plugin>dynamixel_hardware_interface/DynamixelHardware</plugin>
             <param name="port_name">${port_name}</param>
-            <param name="baud_rate">6250000</param>
+            <param name="baud_rate">4000000</param>
             <param name="error_timeout_ms">500</param>
             <param name="dynamixel_model_folder">/param/dxl_model</param>
-            <param name="number_of_joints">6</param>
-            <param name="number_of_transmissions">6</param>
+            <param name="number_of_joints">7</param>
+            <param name="number_of_transmissions">7</param>
             <param name="disable_torque_at_init">true</param>
             <param name="transmission_to_joint_matrix">
-              1, 0, 0, 0, 0, 0,
-              0, 1, 0, 0, 0, 0,
-              0, 0, 1, 0, 0, 0,
-              0, 0, 0, 1, 0, 0,
-              0, 0, 0, 0, 1, 0,
-              0, 0, 0, 0, 0, 1
+              1, 0, 0, 0, 0, 0, 0,
+              0, 1, 0, 0, 0, 0, 0,
+              0, 0, 1, 0, 0, 0, 0,
+              0, 0, 0, 1, 0, 0, 0,
+              0, 0, 0, 0, 1, 0, 0,
+              0, 0, 0, 0, 0, 1, 0,
+              0, 0, 0, 0, 0, 0, 1
             </param>
             <param name="joint_to_transmission_matrix">
-              1, 0, 0, 0, 0, 0,
-              0, 1, 0, 0, 0, 0,
-              0, 0, 1, 0, 0, 0,
-              0, 0, 0, 1, 0, 0,
-              0, 0, 0, 0, 1, 0,
-              0, 0, 0, 0, 0, 1
+              1, 0, 0, 0, 0, 0, 0,
+              0, 1, 0, 0, 0, 0, 0,
+              0, 0, 1, 0, 0, 0, 0,
+              0, 0, 0, 1, 0, 0, 0,
+              0, 0, 0, 0, 1, 0, 0,
+              0, 0, 0, 0, 0, 1, 0,
+              0, 0, 0, 0, 0, 0, 1
             </param>
             <param name="dynamixel_state_pub_msg_name">dynamixel_hardware_interface/dxl_state</param>
@@ -84,4 +86,10 @@
         <state_interface name="effort"/>
       </joint>
+      <joint name="${prefix}rh_r1_joint">
+        <command_interface name="position"/>
+        <state_interface name="position"/>
+        <state_interface name="velocity"/>
+        <state_interface name="effort"/>
+      </joint>
       <gpio name="dxl1">
         <param name="type">dxl</param>
@@ -91,17 +99,12 @@
         <state_interface name="Present Velocity"/>
         <state_interface name="Present Current"/>
-        <param name="Drive Mode">4</param>
-        <param name="Velocity Limit">3591</param>
-        <param name="Acceleration Limit">8050</param>
-        <param name="Profile Velocity">3591</param>
-        <param name="Profile Acceleration">8050</param>
-        <param name="Homing Offset">0</param>
-        <param name="Return Delay Time">0</param>
-        <param name="Position P Gain">1583185</param>
-        <param name="Velocity P Gain">41387</param>
-        <param name="Velocity I Gain">1565630</param>
-        <param name="Operating Mode">3</param>
-        <param name="Profile Acceleration Time">500</param>
-        <param name="Profile Time">1000</param>
+        <param name="Return Delay Time">0</param>
+        <param name="Drive Mode">4</param>
+        <param name="Operating Mode">3</param>
+        <param name="Profile Velocity">10</param>
+        <param name="Profile Acceleration">5</param>
+        <param name="Position P Gain">1000</param>
+        <param name="Position I Gain">0</param>
+        <param name="Position D Gain">200</param>
       </gpio>
       <gpio name="dxl2">
@@ -112,16 +115,12 @@
         <state_interface name="Present Velocity"/>
         <state_interface name="Present Current"/>
+        <param name="Return Delay Time">0</param>
         <param name="Drive Mode">5</param>
-        <param name="Velocity Limit">3591</param>
-        <param name="Acceleration Limit">8050</param>
-        <param name="Profile Velocity">3591</param>
-        <param name="Profile Acceleration">8050</param>
-        <param name="Return Delay Time">0</param>
-        <param name="Position P Gain">1583185</param>
-        <param name="Velocity P Gain">41387</param>
-        <param name="Velocity I Gain">1565630</param>
-        <param name="Operating Mode">3</param>
-        <param name="Profile Acceleration Time">500</param>
-        <param name="Profile Time">1000</param>
+        <param name="Operating Mode">3</param>
+        <param name="Profile Velocity">10</param>
+        <param name="Profile Acceleration">5</param>
+        <param name="Position P Gain">1000</param>
+        <param name="Position I Gain">0</param>
+        <param name="Position D Gain">200</param>
       </gpio>
       <gpio name="dxl3">
@@ -132,16 +131,12 @@
         <state_interface name="Present Velocity"/>
         <state_interface name="Present Current"/>
-        <param name="Drive Mode">4</param>
-        <param name="Velocity Limit">6486</param>
-        <param name="Acceleration Limit">8050</param>
-        <param name="Profile Velocity">6486</param>
-        <param name="Profile Acceleration">8050</param>
-        <param name="Return Delay Time">0</param>
-        <param name="Position P Gain">1583185</param>
-        <param name="Velocity P Gain">18184</param>
-        <param name="Velocity I Gain">1585331</param>
-        <param name="Operating Mode">3</param>
-        <param name="Profile Acceleration Time">500</param>
-        <param name="Profile Time">1000</param>
+        <param name="Return Delay Time">0</param>
+        <param name="Drive Mode">4</param>
+        <param name="Operating Mode">3</param>
+        <param name="Profile Velocity">10</param>
+        <param name="Profile Acceleration">5</param>
+        <param name="Position P Gain">1000</param>
+        <param name="Position I Gain">0</param>
+        <param name="Position D Gain">200</param>
       </gpio>
       <gpio name="dxl4">
@@ -152,16 +147,12 @@
         <state_interface name="Present Velocity"/>
         <state_interface name="Present Current"/>
+        <param name="Return Delay Time">0</param>
         <param name="Drive Mode">5</param>
-        <param name="Velocity Limit">6486</param>
-        <param name="Acceleration Limit">8050</param>
-        <param name="Profile Velocity">6486</param>
-        <param name="Profile Acceleration">8050</param>
-        <param name="Return Delay Time">0</param>
-        <param name="Position P Gain">1583185</param>
-        <param name="Velocity P Gain">18184</param>
-        <param name="Velocity I Gain">1585331</param>
-        <param name="Operating Mode">3</param>
-        <param name="Profile Acceleration Time">500</param>
-        <param name="Profile Time">1000</param>
+        <param name="Operating Mode">3</param>
+        <param name="Profile Velocity">10</param>
+        <param name="Profile Acceleration">5</param>
+        <param name="Position P Gain">1000</param>
+        <param name="Position I Gain">0</param>
+        <param name="Position D Gain">200</param>
       </gpio>
       <gpio name="dxl5">
@@ -172,16 +163,12 @@
         <state_interface name="Present Velocity"/>
         <state_interface name="Present Current"/>
-        <param name="Drive Mode">4</param>
-        <param name="Velocity Limit">6486</param>
-        <param name="Acceleration Limit">8050</param>
-        <param name="Profile Velocity">6486</param>
-        <param name="Profile Acceleration">8050</param>
-        <param name="Return Delay Time">0</param>
-        <param name="Position P Gain">1583185</param>
-        <param name="Velocity P Gain">18184</param>
-        <param name="Velocity I Gain">1585331</param>
-        <param name="Operating Mode">3</param>
-        <param name="Profile Acceleration Time">500</param>
-        <param name="Profile Time">1000</param>
+        <param name="Return Delay Time">0</param>
+        <param name="Drive Mode">4</param>
+        <param name="Operating Mode">3</param>
+        <param name="Profile Velocity">10</param>
+        <param name="Profile Acceleration">5</param>
+        <param name="Position P Gain">1000</param>
+        <param name="Position I Gain">0</param>
+        <param name="Position D Gain">200</param>
       </gpio>
       <gpio name="dxl6">
@@ -192,28 +179,28 @@
         <state_interface name="Present Velocity"/>
         <state_interface name="Present Current"/>
+        <param name="Return Delay Time">0</param>
         <param name="Drive Mode">5</param>
-        <param name="Velocity Limit">6486</param>
-        <param name="Acceleration Limit">8050</param>
-        <param name="Profile Velocity">6486</param>
-        <param name="Profile Acceleration">8050</param>
-        <param name="Return Delay Time">0</param>
-        <param name="Position P Gain">1583185</param>
-        <param name="Velocity P Gain">18184</param>
-        <param name="Velocity I Gain">1585331</param>
-        <param name="Operating Mode">3</param>
-        <param name="Profile Acceleration Time">500</param>
-        <param name="Profile Time">1000</param>
-      </gpio>
-      <gpio name="omy_hat">
-        <param name="type">controller</param>
-        <param name="ID">200</param>
-        <param name="Power Enable">1</param>
-        <param name="Voltage Control Enable">1</param>
-        <param name="R LED">200</param>
-        <param name="G LED">200</param>
-        <param name="B LED">120</param>
-        <param name="Baud Rate (Bus)">8</param>
-        <param name="DXL Baud Rate">8</param>
-        <param name="Status">0</param>
+        <param name="Operating Mode">3</param>
+        <param name="Profile Velocity">10</param>
+        <param name="Profile Acceleration">5</param>
+        <param name="Position P Gain">1000</param>
+        <param name="Position I Gain">0</param>
+        <param name="Position D Gain">200</param>
+      </gpio>
+      <gpio name="dxl7">
+        <param name="type">dxl</param>
+        <param name="ID">7</param>
+        <command_interface name="Goal Position"/>
+        <state_interface name="Present Position"/>
+        <state_interface name="Present Velocity"/>
+        <state_interface name="Present Current"/>
+        <param name="Return Delay Time">0</param>
+        <param name="Drive Mode">4</param>
+        <param name="Operating Mode">3</param>
+        <param name="Profile Velocity">10</param>
+        <param name="Profile Acceleration">5</param>
+        <param name="Position P Gain">1000</param>
+        <param name="Position I Gain">0</param>
+        <param name="Position D Gain">200</param>
       </gpio>
     </ros2_control>

File: urdf/omx_l/omx_l.urdf.xacro (robot description, xacro)
@@ -1,12 +1,12 @@
 <?xml version="1.0"?>
-<robot name="omy_l100" xmlns:xacro="http://www.ros.org/wiki/xacro">
+<robot name="omx_l" xmlns:xacro="http://www.ros.org/wiki/xacro">
   <xacro:arg name="prefix" default="" />
   <xacro:arg name="use_sim" default="false" />
   <xacro:arg name="use_fake_hardware" default="false" />
   <xacro:arg name="fake_sensor_commands" default="false" />
-  <xacro:arg name="port_name" default="/dev/ttyUSB0" />
-  <xacro:arg name="ros2_control_type" default="omy_l100_current" />
-  <xacro:include filename="$(find open_manipulator_description)/urdf/omy_l100/omy_l100_arm.urdf.xacro" />
-  <xacro:include filename="$(find open_manipulator_description)/gazebo/omy_l100.gazebo.xacro" />
+  <xacro:arg name="port_name" default="/dev/ttyACM1" />
+  <xacro:arg name="ros2_control_type" default="omx_l" />
+  <xacro:include filename="$(find open_manipulator_description)/urdf/omx_l/omx_l_arm.urdf.xacro" />
+  <xacro:include filename="$(find open_manipulator_description)/gazebo/omx_l.gazebo.xacro" />
   <xacro:include filename="$(find open_manipulator_description)/ros2_control/$(arg ros2_control_type).ros2_control.xacro" />
   <link name="world"/>
@@ -16,8 +16,8 @@
     <origin xyz="0.0 0.0 0.0" rpy="0 0 0"/>
   </joint>
-  <xacro:omy_l100 prefix="$(arg prefix)" />
-  <xacro:omy_l100_gazebo prefix="$(arg prefix)" />
-  <xacro:omy_l100_system
-    name="OMYL100System" prefix="$(arg prefix)" use_sim="$(arg use_sim)"
+  <xacro:omx_l prefix="$(arg prefix)" />
+  <xacro:omx_l_gazebo prefix="$(arg prefix)" />
+  <xacro:omx_l_system
+    name="OMXLEADERSYSTEM" prefix="$(arg prefix)" use_sim="$(arg use_sim)"
     use_fake_hardware="$(arg use_fake_hardware)"
     fake_sensor_commands="$(arg fake_sensor_commands)"
@@ -25,5 +25,5 @@
   <gazebo>
     <plugin filename="gz_ros2_control-system" name="gz_ros2_control::GazeboSimROS2ControlPlugin">
-      <parameters>$(find open_manipulator_bringup)/config/om_y_leader/gazebo_controller_manager.yaml</parameters>
+      <parameters>$(find open_manipulator_bringup)/config/omx_l_leader/hardware_controller_manager.yaml</parameters>
     </plugin>
   </gazebo>
