Commit message: Rebase from 'upstream'

File: open_manipulator_description/urdf/omy_f3m/omy_f3m.urdf (robot description, URDF)
Before this commit: robot omy_f3m, 15 links, 14 joints
Links:
- added link camera_bottom_screw_frame
- added link camera_link, mass 0.072; collision box size=0.023 0.042 0.042; visual mesh filename=package://realsense2_description/meshes/d405.stl scale=0.001 0.001 0.001
Joints:
- added joint camera_joint: type fixed, parent link6, child camera_bottom_screw_frame, origin xyz=-0.021 -0.07385 0.0803 rpy=-1.57079632679 0 -1.57079632679
- added joint camera_link_joint: type fixed, parent camera_bottom_screw_frame, child camera_link, origin xyz=0.01085 0.009 0.021 rpy=0 0 0

File: open_manipulator_description/urdf/omy_f3m/omy_f3m_arm.urdf.xacro (robot description, xacro)
@@ -2,4 +2,5 @@
 <robot xmlns:xacro="http://www.ros.org/wiki/xacro">
    <xacro:macro name="omy_f3m" params="prefix">
+      <xacro:include filename="$(find realsense2_description)/urdf/_d405.urdf.xacro" />
       <xacro:property name="meshes_file_direction" value="package://open_manipulator_description/meshes/omy_f3m" />
       <link name="${prefix}link0">
@@ -205,4 +206,7 @@
          </inertial>
       </link>
+      <xacro:sensor_d405 parent="${prefix}link6" use_nominal_extrinsics="false" name="${prefix}camera">
+         <origin xyz="-0.021 -0.07385 0.0803" rpy="-1.57079632679 0 -1.57079632679"/>
+      </xacro:sensor_d405>
       <joint name="${prefix}end_effector_flange_joint" type="fixed">
          <parent link="${prefix}link6" />

Commit message: Imported upstream version '4.1.2' of 'upstream'

File: open_manipulator_description/urdf/omy_f3m/omy_f3m.urdf (robot description, URDF)
Before this commit: robot omy_f3m, 17 links, 16 joints
Links:
- removed link camera_bottom_screw_frame
- removed link camera_link
Joints:
- removed joint camera_joint
- removed joint camera_link_joint

File: open_manipulator_description/urdf/omy_f3m/omy_f3m_arm.urdf.xacro (robot description, xacro)
@@ -2,5 +2,4 @@
 <robot xmlns:xacro="http://www.ros.org/wiki/xacro">
    <xacro:macro name="omy_f3m" params="prefix">
-      <xacro:include filename="$(find realsense2_description)/urdf/_d405.urdf.xacro" />
       <xacro:property name="meshes_file_direction" value="package://open_manipulator_description/meshes/omy_f3m" />
       <link name="${prefix}link0">
@@ -206,7 +205,4 @@
          </inertial>
       </link>
-      <xacro:sensor_d405 parent="${prefix}link6" use_nominal_extrinsics="false" name="${prefix}camera">
-         <origin xyz="-0.021 -0.07385 0.0803" rpy="-1.57079632679 0 -1.57079632679"/>
-      </xacro:sensor_d405>
       <joint name="${prefix}end_effector_flange_joint" type="fixed">
          <parent link="${prefix}link6" />
